File: PCB/totem_0-3/totem_0_3.kicad_sch (KiCad schematic)
At the start: 80 parts, among them J1 MJ-4PP-9, J2 MJ-4PP-9, U1 xiao-RP2040, U2 xiao-rp2040

Commit message: Fully wired
Parts:
- U1: value xiao-RP2040 -> xiao-rp2040
Connections:
- net COL0_L: now also U1.2 (A1/D1); no longer U1.5 (A8_SDA/0.04_H)
- net COL1_L: now also U1.1 (A0/D0); no longer U1.6 (A9_SCL/0.05_H)
- net ROW0_L: now also U1.6 (SCL/D5); no longer U1.1 (A2/0.02_H)
- net ROW1_L: now also U1.5 (SDA/D4); no longer U1.2 (A4/0.03_H)
- net ROW2_L: now also U1.4 (A3/D3); no longer U1.3 (A10/0.28)
- net ROW3_L: now also U1.3 (A2/D2); no longer U1.4 (A11/0.29)
