File: pcb/fabiTEM.kicad_sch (KiCad schematic)
At the start: 116 parts, among them J1 USB_C_Receptacle_USB2.0_14P, J2 USB_C_Receptacle_USB2.0_14P, J3 USB_C_Receptacle_USB2.0_14P, U1 AP2112K-3.3, U2 RP2040, U3 W25Q16JVSSIQ, U5 MCP23017-EML, Y1 ABM8-272-T3

Commit message: 0.8
Parts:
- removed J2: USB_C_Receptacle_USB2.0_14P, fabiTEM:USB_C_Receptacle_GCT_USB4105-xx-A_16P_TopMnt_Horizontal, symbol fabiTEM:USB_C_Receptacle_USB2.0_14P
- added J2: TYPE-C16PIN, fabiTEM:USB_C_Receptacle_GCT_USB4105-xx-A_16P_MidMnt_Horizontal, symbol fabiTEM:USB_C_Receptacle_USB2.0_16P
- J1, J3: value USB_C_Receptacle_USB2.0_14P -> TYPE-C16PIN; footprint fabiTEM:USB_C_Receptacle_GCT_USB4105-xx-A_16P_TopMnt_Horizontal -> fabiTEM:USB_C_Receptacle_GCT_USB4105-xx-A_16P_MidMnt_Horizontal; symbol fabiTEM:USB_C_Receptacle_USB2.0_14P -> fabiTEM:USB_C_Receptacle_USB2.0_16P
Connections:
- net D+: now also J2.A6 (D+), J2.B6 (D+)
- net D-: now also J2.A7 (D-), J2.B7 (D-)
- net GND: now also J2.A1 (GND), J2.A12 (GND), J2.B1 (GND), J2.B12 (GND), J2.S1 (SHIELD)
- net at R10.1: now also J2.B5 (CC2)
- net at R9.1: now also J2.A5 (CC1)
- net at D1.2: now also J2.A4 (VBUS), J2.A9 (VBUS), J2.B4 (VBUS), J2.B9 (VBUS)
- no-connect marks 23 -> 29
